Commit message: fix: use measured drivetrain geometry

File: ros2_ws/src/botix_description/urdf/botix.urdf (robot description, URDF)
Before this commit: robot botix, 11 links, 10 joints
Links:
- link left_wheel_link: geometry collision cylinder length=0.0254 radius=0.0335; visual cylinder length=0.0254 radius=0.0335
- link right_wheel_link: geometry collision cylinder length=0.0254 radius=0.0335; visual cylinder length=0.0254 radius=0.0335
Joints:
- joint base_footprint_to_base_link: origin xyz=0 0 0.0338 rpy=0 0 0 -> xyz=0 0 0.0335 rpy=0 0 0
- joint left_wheel_joint: origin xyz=0.000 0.0877 0.000 rpy=0 0 0 -> xyz=0.000 0.0875 0.000 rpy=0 0 0
- joint right_wheel_joint: origin xyz=0.000 -0.0877 0.000 rpy=0 0 0 -> xyz=0.000 -0.0875 0.000 rpy=0 0 0
